File: NegiCon/NegiCon.kicad_pcb (KiCad board)
At the start: 2 copper layers, 41 parts, among them U1 LM1117MP-3.3, U4 SC0915

Commit message: add connectors for air sensors
Parts:
- added J1: Left Air Sensor, Connector_Molex:Molex_Nano-Fit_105313-xx04_1x04_P2.50mm_Horizontal, F.Cu at (56.2, 319.0)
- added J2: Right Air Sensor, Connector_Molex:Molex_Nano-Fit_105313-xx04_1x04_P2.50mm_Horizontal, F.Cu at (547.9, 314.2)
- U4: value SC0915 -> Pi Pico
Connections:
- U4 pad 19: unconnected-(U4-GP14-Pad19) -> SDA_air
- U4 pad 20: unconnected-(U4-GP15-Pad20) -> SCL_air
