File: openithm-new/main.kicad_sch (KiCad schematic)
At the start: 22 parts, among them SW1 SW_Push, SW2 SW_SPDT, U1 STM32F072VBTx, Y1 48MHz, 7pF

Commit message: Finished Rev.1
Parts:
- removed C11, C12: 4p, Capacitor_SMD:C_0402_1005Metric, symbol Device:C_Small
- removed R1: 10k, Resistor_SMD:R_0402_1005Metric, symbol Device:R_Small_US
- removed SW2: SW_SPDT, Button_Switch_SMD:SW_SPDT_PCM12, symbol Switch:SW_SPDT
- removed Y1: 48MHz, 7pF, Crystal:Crystal_SMD_3225-4Pin_3.2x2.5mm, symbol Device:Crystal_GND24
- added R3: 10k, Resistor_SMD:R_0402_1005Metric, symbol Device:R_Small_US
- added SW2: SW_Push, Button_Switch_SMD:SW_Tactile_SPST_NO_Straight_CK_PTS636Sx25SMTRLFS, symbol Switch:SW_Push
- H1, H2, H3, H4: footprint MountingHole:MountingHole_2.2mm_M2_Pad_Via -> MountingHole:MountingHole_2.2mm_M2_Pad
Connections:
- net +3.3V: now also SW2.1
- net GND: now also R3.1; no longer H1.1, H2.1, H3.1, H4.1
- net BOOT0: now reaches U1.94 (BOOT0)
- net BOOT0: now also R3.2, SW2.2
- net HSE_IN: no longer names the net of U1.12 (PF0)
- net HSE_OUT: no longer names the net of U1.13 (PF1)
- net I2C1_SCL: no longer names the net of U1.95 (PB8)
- net I2C1_SDA: no longer names the net of U1.96 (PB9)
- no-connect marks 6 -> 12
