File: openithm-new/main_conn.kicad_sch (KiCad schematic)
At the start: 3 parts, among them J1 I2C1, J2 USB_B_Micro, J3 Touch Control Connector

Commit message: Finished Rev.1
Parts:
- removed J1: I2C1, Connector_PinHeader_2.54mm:PinHeader_1x02_P2.54mm_Vertical, symbol Connector:Conn_01x02_Socket
- removed J3: Touch Control Connector, Connector_JST:JST_PHD_S24B-PHDSS_2x12_P2.00mm_Horizontal, symbol Connector_Generic:Conn_02x12_Top_Bottom
- added J3: SW Debug, Connector_PinHeader_2.54mm:PinHeader_1x04_P2.54mm_Horizontal, symbol Connector:Conn_01x04_Pin
Connections:
- net GND: now also J3.4 (Pin_4)
- new net +3.3V: J3.1 (Pin_1)
- new net SWCLK: J3.3 (Pin_3)
- new net SWDIO: J3.2 (Pin_2)
Changed lines of the file:
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@@
+	(wire
+		(pts
+			(xy 96.52 59.69) (xy 101.6 59.69)
+		)
+		(stroke
+			(width 0)
+			(type default)
+		)
+	)
+	(wire
+		(pts
+			(xy 101.6 59.69) (xy 101.6 62.23)
+		)
+		(stroke
+			(width 0)
+			(type default)
+		)
+	)
 	(wire
 		(pts
@@
 	(wire
 		(pts
+			(xy 101.6 52.07) (xy 96.52 52.07)
+		)
+		(stroke
+			(width 0)
+			(type default)
+		)
+	)
+	(wire
+		(pts
 			(xy 45.72 62.23) (xy 45.72 59.69)
 		)
@@
 		(pts
 			(xy 53.34 44.45) (xy 63.5 44.45)
+		)
+		(stroke
+			(width 0)
+			(type default)
+		)
+	)
+	(wire
+		(pts
+			(xy 101.6 49.53) (xy 101.6 52.07)
 		)
 		(stroke
@@
 		)
 	)
-	(global_label "I2C1_SCL"
+	(global_label "SWCLK"
 		(shape input)
-		(at 144.78 38.1 0)
+		(at 96.52 57.15 0)
 		(fields_autoplaced yes)
 		(effects
@@
 		)
 		(property "Intersheetrefs" "${INTERSHEET_REFS}"
-			(at 156.5342 38.1 0)
+			(at 105.7342 57.15 0)
 			(effects
 				(font
@@
 		)
 	)
-	(global_label "I2C1_SDA"
+	(global_label "SWDIO"
 		(shape input)
-		(at 144.78 40.64 0)
+		(at 96.52 54.61 0)
 		(fields_autoplaced yes)
 		(effects
@@
 		)
 		(property "Intersheetrefs" "${INTERSHEET_REFS}"
-			(at 156.5947 40.64 0)
+			(at 105.3714 54.61 0)
 			(effects
 				(font
@@
 	)
 	(symbol
-		(lib_id "Connector:Conn_01x02_Socket")
-		(at 139.7 38.1 0)
-		(mirror y)
+		(lib_id "power:+3.3V")
+		(at 101.6 49.53 0)
 		(unit 1)
 		(exclude_from_sim no)
@@
 		(dnp no)
 		(fields_autoplaced yes)
-		(property "Reference" "J1"
-			(at 138.43 38.0999 0)
-			(effects
-				(font
-					(size 1.27 1.27)
-				)
-				(justify left)
-			)
-		)
-		(property "Value" "I2C1"
-			(at 138.43 40.6399 0)
-			(effects
-				(font
-					(size 1.27 1.27)
-				)
-				(justify left)
-			)
-		)
-		(property "Footprint" "Connector_PinHeader_2.54mm:PinHeader_1x02_P2.54mm_Vertical"
-			(at 139.7 38.1 0)
-			(effects
-				(font
-					(size 1.27 1.27)
-				)
-				(hide yes)
-			)
-		)
-		(property "Datasheet" "~"
-			(at 139.7 38.1 0)
-			(effects
-				(font
-					(size 1.27 1.27)
-				)
-				(hide yes)
-			)
-		)
-		(property "Description" "Generic connector, single row, 01x02, script generated"
-			(at 139.7 38.1 0)
-			(effects
-				(font
-					(size 1.27 1.27)
-				)
-				(hide yes)
-			)
-		)
-		(pin "2"
+		(property "Reference" "#PWR010"
+			(at 101.6 53.34 0)
+			(effects
+				(font
+					(size 1.27 1.27)
+				)
+				(hide yes)
+			)
+		)
+		(property "Value" "+3.3V"
+			(at 101.6 44.45 0)
+			(effects
+				(font
+					(size 1.27 1.27)
+				)
+			)
+		)
+		(property "Footprint" ""
+			(at 101.6 49.53 0)
+			(effects
+				(font
+					(size 1.27 1.27)
+				)
+				(hide yes)
+			)
+		)
+		(property "Datasheet" ""
+			(at 101.6 49.53 0)
+			(effects
+				(font
+					(size 1.27 1.27)
+				)
+				(hide yes)
+			)
+		)
+		(property "Description" "Power symbol creates a global label with name \"+3.3V\""
+			(at 101.6 49.53 0)
+			(effects
+				(font
+					(size 1.27 1.27)
+				)
+				(hide yes)
+			)
 		)
 		(pin "1"
 		)
 		(instances
-			(project ""
+			(project "openithm-new"
 				(path "/24ef4980-772f-43bd-95fe-2a56cd9ca729/0bc1cbc6-7225-43f6-987e-178a5cf4a396/19f89589-6976-49b1-8e8a-80c19b06dfbf"
-					(reference "J1")
+					(reference "#PWR010")
 					(unit 1)
 				)
@@
 	)
 	(symbol
+		(lib_id "Connector:Conn_01x04_Pin")
+		(at 91.44 54.61 0)
+		(unit 1)
+		(exclude_from_sim no)
+		(in_bom yes)
+		(on_board yes)
+		(dnp no)
+		(fields_autoplaced yes)
+		(property "Reference" "J3"
+			(at 92.075 46.99 0)
+			(effects
+				(font
+					(size 1.27 1.27)
+				)
+			)
+		)
+		(property "Value" "SW Debug"
+			(at 92.075 49.53 0)
+			(effects
+				(font
+					(size 1.27 1.27)
+				)
+			)
+		)
+		(property "Footprint" "Connector_PinHeader_2.54mm:PinHeader_1x04_P2.54mm_Horizontal"
+			(at 91.44 54.61 0)
+			(effects
+				(font
+					(size 1.27 1.27)
+				)
+				(hide yes)
+			)
+		)
+		(property "Datasheet" "~"
+			(at 91.44 54.61 0)
+			(effects
+				(font
+					(size 1.27 1.27)
+				)
+				(hide yes)
+			)
+		)
+		(property "Description" "Generic connector, single row, 01x04, script generated"
+			(at 91.44 54.61 0)
+			(effects
+				(font
+					(size 1.27 1.27)
+				)
+				(hide yes)
+			)
+		)
+		(pin "4"
+		)
+		(pin "2"
+		)
+		(pin "1"
+		)
+		(pin "3"
+		)
+		(instances
+			(project ""
+				(path "/24ef4980-772f-43bd-95fe-2a56cd9ca729/0bc1cbc6-7225-43f6-987e-178a5cf4a396/19f89589-6976-49b1-8e8a-80c19b06dfbf"
+					(reference "J3")
+					(unit 1)
+				)
+			)
+		)
+	)
+	(symbol
 		(lib_id "Connector:USB_B_Micro")
 		(at 45.72 49.53 0)
@@
 	)
 	(symbol
-		(lib_id "Connector_Generic:Conn_02x12_Top_Bottom")
-		(at 97.79 52.07 0)
+		(lib_id "power:GND")
+		(at 101.6 62.23 0)
 		(unit 1)
 		(exclude_from_sim no)
@@
 		(dnp no)
 		(fields_autoplaced yes)
-		(property "Reference" "J3"
-			(at 99.06 33.02 0)
-			(effects
-				(font
-					(size 1.27 1.27)
-				)
-			)
-		)
-		(property "Value" "Touch Control Connector"
-			(at 99.06 35.56 0)
-			(effects
-				(font
-					(size 1.27 1.27)
-				)
-			)
-		)
-		(property "Footprint" "Connector_JST:JST_PHD_S24B-PHDSS_2x12_P2.00mm_Horizontal"
-			(at 97.79 52.07 0)
-			(effects
-				(font
-					(size 1.27 1.27)
-				)
-				(hide yes)
-			)
-		)
-		(property "Datasheet" "~"
-			(at 97.79 52.07 0)
-			(effects
-				(font
-					(size 1.27 1.27)
-				)
-				(hide yes)
-			)
-		)
-		(property "Description" "Generic connector, double row, 02x12, top/bottom pin numbering scheme (row 1: 1...pins_per_row, row2: pins_per_row+1 ... num_pins), script generated (kicad-library-utils/schlib/autogen/connector/)"
-			(at 97.79 52.07 0)
-			(effects
-				(font
-					(size 1.27 1.27)
-				)
-				(hide yes)
-			)
-		)
-		(pin "17"
-		)
-		(pin "12"
-		)
-		(pin "13"
-		)
-		(pin "2"
-		)
-		(pin "7"
-		)
-		(pin "24"
-		)
-		(pin "15"
-		)
-		(pin "6"
-		)
-		(pin "9"
-		)
-		(pin "16"
-		)
-		(pin "14"
-		)
-		(pin "21"
-		)
-		(pin "22"
-		)
-		(pin "3"
-		)
-		(pin "20"
-		)
-		(pin "10"
-		)
-		(pin "23"
-		)
-		(pin "11"
+		(property "Reference" "#PWR021"
+			(at 101.6 68.58 0)
+			(effects
+				(font
+					(size 1.27 1.27)
+				)
+				(hide yes)
+			)
+		)
+		(property "Value" "GND"
+			(at 101.6 67.31 0)
+			(effects
+				(font
+					(size 1.27 1.27)
+				)
+			)
+		)
+		(property "Footprint" ""
+			(at 101.6 62.23 0)
+			(effects
+				(font
+					(size 1.27 1.27)
+				)
+				(hide yes)
+			)
+		)
+		(property "Datasheet" ""
+			(at 101.6 62.23 0)
+			(effects
+				(font
+					(size 1.27 1.27)
+				)
+				(hide yes)
+			)
+		)
+		(property "Description" "Power symbol creates a global label with name \"GND\" , ground"
+			(at 101.6 62.23 0)
+			(effects
+				(font
+					(size 1.27 1.27)
+				)
+				(hide yes)
+			)
 		)
 		(pin "1"
 		)
-		(pin "19"
-		)
-		(pin "4"
-		)
-		(pin "18"
-		)
-		(pin "8"
-		)
-		(pin "5"
-		)
 		(instances
-			(project ""
+			(project "openithm-new"
 				(path "/24ef4980-772f-43bd-95fe-2a56cd9ca729/0bc1cbc6-7225-43f6-987e-178a5cf4a396/19f89589-6976-49b1-8e8a-80c19b06dfbf"
-					(reference "J3")
+					(reference "#PWR021")
 					(unit 1)
 				)
