File: openithm-new/openithm-new.kicad_pcb (KiCad board)
At the start: 2 copper layers, 30 parts, among them J1 I2C1, J2 USB_B_Micro, J3 Touch Control Connector, SW1 SW_Push, SW2 SW_SPDT, U1 STM32F072VBTx, U2 TLV76733DRVR, Y1 48MHz, 7pF

Commit message: Finished Rev.1
Parts:
- removed J1: I2C1, Connector_PinHeader_2.54mm:PinHeader_1x02_P2.54mm_Vertical
- removed Y1: 48MHz, 7pF, Crystal:Crystal_SMD_3225-4Pin_3.2x2.5mm
- added C15: 4n7, Capacitor_SMD:C_0402_1005Metric, F.Cu at (421.3, 255.7)
- added C16: 4n7, Capacitor_SMD:C_0402_1005Metric, F.Cu at (424.9, 254.1)
- added C17: 4n7, Capacitor_SMD:C_0402_1005Metric, F.Cu at (427.9, 250.3)
- added C18: 4n7, Capacitor_SMD:C_0402_1005Metric, F.Cu at (430.0, 248.3)
- added J4: AC Slider, Openithm:AC_SLIDER, F.Cu at (420.4, 314.6)
- added R10: 1k, Resistor_SMD:R_0402_1005Metric, F.Cu at (419.6, 255.6)
- added R11: 1k, Resistor_SMD:R_0402_1005Metric, F.Cu at (427.5, 256.2)
- added R12: 1k, Resistor_SMD:R_0402_1005Metric, F.Cu at (428.4, 255.4)
- added R13: 1k, Resistor_SMD:R_0402_1005Metric, F.Cu at (429.2, 254.6)
- added R14: 1k, Resistor_SMD:R_0402_1005Metric, F.Cu at (430.1, 253.7)
- added R15: 1k, Resistor_SMD:R_0402_1005Metric, F.Cu at (430.9, 252.9)
- added R16: 1k, Resistor_SMD:R_0402_1005Metric, F.Cu at (431.8, 252.0)
- added R17: 1k, Resistor_SMD:R_0402_1005Metric, F.Cu at (432.3, 242.6)
- added R18: 1k, Resistor_SMD:R_0402_1005Metric, F.Cu at (432.7, 241.3)
- added R3: 10k, Resistor_SMD:R_0402_1005Metric, F.Cu at (395.3, 235.2)
- added R4: 1k, Resistor_SMD:R_0402_1005Metric, F.Cu at (411.1, 238.8)
- added R5: 1k, Resistor_SMD:R_0402_1005Metric, F.Cu at (409.6, 247.4)
- added R6: 1k, Resistor_SMD:R_0402_1005Metric, F.Cu at (410.3, 248.1)
- added R7: 1k, Resistor_SMD:R_0402_1005Metric, F.Cu at (411.1, 248.8)
- added R8: 1k, Resistor_SMD:R_0402_1005Metric, F.Cu at (417.1, 254.6)
- added R9: 1k, Resistor_SMD:R_0402_1005Metric, F.Cu at (417.9, 255.3)
- C11, C12: value 4p -> 4n7
- H1, H2, H3, H4: footprint MountingHole:MountingHole_2.2mm_M2_Pad_Via -> MountingHole:MountingHole_2.2mm_M2_Pad
- J3: value Touch Control Connector -> SW Debug; footprint Connector_JST:JST_PHD_S24B-PHDSS_2x12_P2.00mm_Horizontal -> Connector_PinHeader_2.54mm:PinHeader_1x04_P2.54mm_Horizontal
- R1: value 10k -> 1k
- SW2: value SW_SPDT -> SW_Push; footprint Button_Switch_SMD:SW_SPDT_PCM12 -> Button_Switch_SMD:SW_Tactile_SPST_NO_Straight_CK_PTS636Sx25SMTRLFS
- moved H2 631.9 mm to (650.5, 363.5), turned to 180 degrees
- moved H1 518.0 mm to (650.5, 263.5), turned to 180 degrees
- moved C4 349.8 mm to (432.8, 247.8), turned to -135 degrees
- moved C2 349.1 mm to (423.4, 254.9), turned to -135 degrees
- moved C3 346.5 mm to (431.5, 246.8), turned to -135 degrees
- moved C7 343.6 mm to (415.7, 253.3), turned to 135 degrees
- moved C9 343.1 mm to (412.0, 255.4), turned to 45 degrees
- moved FB1 342.2 mm to (413.1, 256.6), turned to 45 degrees
- moved C8 341.0 mm to (414.4, 254.2), turned to 135 degrees
- moved C10 336.1 mm to (413.3, 250.7), turned to -45 degrees
- moved U1 329.8 mm to (420.5, 244.1), turned to 45 degrees
- moved C12 327.8 mm to (409.1, 245.8), turned to 135 degrees
- moved D1 326.8 mm to (431.7, 235.2)
- moved R2 326.1 mm to (432.5, 237.1), turned to -90 degrees
- moved C13 325.6 mm to (433.9, 232.0), turned to -90 degrees
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Connections:
- C11 pad 1: /Main Board/HSE_IN -> TSC_G5_IO1
- C12 pad 1: /Main Board/HSE_OUT -> TSC_G7_IO1
- H1 pad 1: GND -> unconnected-(H1-Pad1)
- H2 pad 1: GND -> unconnected-(H2-Pad1)
- H3 pad 1: GND -> unconnected-(H3-Pad1)
- H4 pad 1: GND -> unconnected-(H4-Pad1)
- J3 pad 1: unconnected-(J3-Pin_1-Pad1) -> +3.3V
- J3 pad 2: unconnected-(J3-Pin_2-Pad2) -> SWDIO
- J3 pad 3: unconnected-(J3-Pin_3-Pad3) -> SWCLK
- J3 pad 4: unconnected-(J3-Pin_4-Pad4) -> GND
- R1 pad 1: Net-(SW2-B) -> Net-(J4-Pin_1)
- R1 pad 2: Net-(U1-BOOT0) -> TSC_G5_IO2
- SW2 pad 1: GND -> +3.3V
- SW2 pad 2: Net-(SW2-B) -> BOOT0
- U1 pad 12: /Main Board/HSE_IN -> unconnected-(U1-PF0-Pad12)
- U1 pad 13: /Main Board/HSE_OUT -> unconnected-(U1-PF1-Pad13)
- U1 pad 94: Net-(U1-BOOT0) -> BOOT0
- U1 pad 95: I2C1_SCL -> unconnected-(U1-PB8-Pad95)
- U1 pad 96: I2C1_SDA -> unconnected-(U1-PB9-Pad96)
Routing:
- net Net-(J4-Pin_1): track 0.00 -> 262.8 mm
- net Net-(J4-Pin_16): track 0.00 -> 250.5 mm
- net Net-(J4-Pin_2): track 0.00 -> 232.8 mm
- net Net-(J4-Pin_15): track 0.00 -> 221.3 mm
- net Net-(J4-Pin_3): track 0.00 -> 192.8 mm
- net Net-(J4-Pin_14): track 0.00 -> 189.0 mm
- net Net-(J4-Pin_4): track 0.00 -> 164.1 mm
- net Net-(J4-Pin_13): track 0.00 -> 160.5 mm
- net Net-(J4-Pin_5): track 0.00 -> 135.3 mm
- net Net-(J4-Pin_12): track 0.00 -> 131.9 mm
- net Net-(J4-Pin_6): track 0.00 -> 108.9 mm
- net Net-(J4-Pin_11): track 0.00 -> 103.4 mm
- net Net-(J4-Pin_7): track 0.00 -> 80.3 mm
- net Net-(J4-Pin_10): track 0.00 -> 75.0 mm
- net +3.3V: track 0.00 -> 72.2 mm, vias 0 -> 11
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- added copper zone on B.Cu, net +3.3V
- added copper zone on F.Cu, net +3.3V
- added copper zone on B.Cu, net GND
- added copper zone on F.Cu, net GND
- added copper zone on F.Cu, net VBUS
Other:
- board outline added: 480 x 155 mm
- board text added: "BOOT0"
- board text added: "GROUND SLIDER"
- board text added: "NRST"
