File: openithm-new/openithm-new.kicad_sch (KiCad schematic)
At the start: 0 parts

Commit message: Finished Rev.1
Other:
- removed sheet Air Sensor IR
- removed sheet Air Sensor Receiver
Changed lines of the file:
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@@
 	)
 	(sheet
-		(at 74.93 49.53)
+		(at 69.85 81.28)
 		(size 74.93 43.18)
 		(fields_autoplaced yes)
@@
 		)
 		(property "Sheetname" "Main Board"
-			(at 74.93 48.8184 0)
+			(at 69.85 80.5684 0)
 			(effects
 				(font
@@
 		)
 		(property "Sheetfile" "main.kicad_sch"
-			(at 74.93 93.2946 0)
+			(at 69.85 125.0446 0)
 			(effects
 				(font
@@
 	)
 	(sheet
-		(at 74.93 102.87)
-		(size 74.93 43.18)
-		(fields_autoplaced yes)
-		(stroke
-			(width 0.1524)
-			(type solid)
-		)
-		(fill
-			(color 0 0 0 0.0000)
-		)
-		(property "Sheetname" "Air Sensor IR"
-			(at 74.93 102.1584 0)
-			(effects
-				(font
-					(size 1.27 1.27)
-				)
-				(justify left bottom)
-			)
-		)
-		(property "Sheetfile" "air_ir.kicad_sch"
-			(at 74.93 146.6346 0)
-			(effects
-				(font
-					(size 1.27 1.27)
-				)
-				(justify left top)
-			)
-		)
-		(instances
-			(project "openithm-new"
-				(path "/24ef4980-772f-43bd-95fe-2a56cd9ca729"
-					(page "4")
-				)
-			)
-		)
-	)
-	(sheet
-		(at 156.21 102.87)
-		(size 74.93 43.18)
-		(fields_autoplaced yes)
-		(stroke
-			(width 0.1524)
-			(type solid)
-		)
-		(fill
-			(color 0 0 0 0.0000)
-		)
-		(property "Sheetname" "Air Sensor Receiver"
-			(at 156.21 102.1584 0)
-			(effects
-				(font
-					(size 1.27 1.27)
-				)
-				(justify left bottom)
-			)
-		)
-		(property "Sheetfile" "air_rec.kicad_sch"
-			(at 156.21 146.6346 0)
-			(effects
-				(font
-					(size 1.27 1.27)
-				)
-				(justify left top)
-			)
-		)
-		(instances
-			(project "openithm-new"
-				(path "/24ef4980-772f-43bd-95fe-2a56cd9ca729"
-					(page "5")
-				)
-			)
-		)
-	)
-	(sheet
-		(at 156.21 49.53)
+		(at 151.13 81.28)
 		(size 74.93 41.91)
 		(fields_autoplaced yes)
@@
 		)
 		(property "Sheetname" "Touch Board"
-			(at 156.21 48.8184 0)
+			(at 151.13 80.5684 0)
 			(effects
 				(font
@@
 		)
 		(property "Sheetfile" "touch.kicad_sch"
-			(at 156.21 92.0246 0)
+			(at 151.13 123.7746 0)
 			(effects
 				(font
