File: openithm-new/touch.kicad_sch (KiCad schematic)
At the start: 0 parts

Commit message: Finished Rev.1
Parts:
- added C11, C12, C15, C16, C17, C18: 4n7, Capacitor_SMD:C_0402_1005Metric, symbol Device:C_Small
- added J4: AC Slider, Openithm:AC_SLIDER, symbol Connector:Conn_01x16_Pin
- added R1, R10, R11, R12, R13, R14, R15, R16, R17, R18, R4, R5, R6, R7, R8, R9: 1k, Resistor_SMD:R_0402_1005Metric, symbol Device:R_Small_US
Connections:
- new net: J4.1 (Pin_1), R1.1
- new net: J4.10 (Pin_10), R12.1
- new net: J4.11 (Pin_11), R13.1
- new net: J4.12 (Pin_12), R14.1
- new net: J4.13 (Pin_13), R15.1
- new net: J4.14 (Pin_14), R16.1
- new net: J4.15 (Pin_15), R17.1
- new net: J4.16 (Pin_16), R18.1
- new net: J4.2 (Pin_2), R4.1
- new net: J4.3 (Pin_3), R5.1
- new net: J4.4 (Pin_4), R6.1
- new net: J4.5 (Pin_5), R7.1
- new net: J4.6 (Pin_6), R8.1
- new net: J4.7 (Pin_7), R9.1
- new net: J4.8 (Pin_8), R10.1
- new net: J4.9 (Pin_9), R11.1
- new net GND: C11.2, C12.2, C15.2, C16.2, C17.2, C18.2
- new net TSC_G1_IO1: R8.2
- new net TSC_G1_IO2: R9.2
- new net TSC_G1_IO3: R10.2
- new net TSC_G1_IO4: C15.1
- new net TSC_G2_IO1: C16.1
- new net TSC_G2_IO2: R11.2
- new net TSC_G2_IO3: R12.2
- new net TSC_G2_IO4: R13.2
- new net TSC_G3_IO1: R14.2
- new net TSC_G3_IO2: R15.2
- new net TSC_G3_IO3: R16.2
- new net TSC_G3_IO4: C17.1
- new net TSC_G5_IO1: C11.1
- new net TSC_G5_IO2: R1.2
- new net TSC_G5_IO3: R4.2
- new net TSC_G6_IO1: C18.1
- new net TSC_G6_IO2: R17.2
- new net TSC_G6_IO3: R18.2
- new net TSC_G7_IO1: C12.1
- new net TSC_G7_IO2: R5.2
- new net TSC_G7_IO3: R6.2
- new net TSC_G7_IO4: R7.2
- no-connect marks 0 -> 2
Other:
- note added: "Sampling Capacitor: 47 n ESD Protection: 1 k C_{Sshield}=k * C_{Skey}, k=A_{shield} / A_{key} A_{key} = 25.5mm * 82mm"
